Commit message: continue building urdf

File: table_description/urdf/table.urdf.xacro (robot description, xacro)
@@ -4,4 +4,5 @@
   <xacro:property name="rod_length" value="${props['rod_length']}"/>
   <xacro:property name="rod_diameter" value="${props['rod_diameter']}"/>
+  <xacro:property name="rod_mountingheight" value="${props['rod_mountingheight']}"/>
   <xacro:property name="player_width" value="${props['player_width']}"/>
   <xacro:property name="player_depth" value="${props['player_depth']}"/>
@@ -10,9 +11,11 @@
   <xacro:property name="field_width" value="${props['field_width']}"/>
   <xacro:property name="field_length" value="${props['field_length']}"/>
+  <xacro:property name="field_thickness" value="0.005"/>
   <xacro:property name="goal_width" value="${props['goal_width']}"/>
   <xacro:property name="goal_height" value="${props['goal_height']}"/>
   <xacro:property name="wall_height" value="${props['wall_height']}"/>
+  <xacro:property name="attack_rod_distance" value="${props['attack_rod_distance']}"/>
+  <xacro:property name="goalie_rod_distance" value="${props['goalie_rod_distance']}"/>
   <xacro:property name="wall_thickness" value="0.015"/>
-  <xacro:property name="field_thickness" value="0.005"/>
   <!-- Macro to create a player -->
   <xacro:macro name="player" params="name r g b">
@@ -28,21 +31,99 @@
   </xacro:macro>
   <!-- Macro to create a player rod -->
-  <xacro:macro name="player_rod" params="name r g b">
-    <link name="${name}">
+  <xacro:macro name="player_rod" params="name dir dist num_players r g b">
+    <link name="${name}_mount_c">
+      <origin xyz="0 0 0" rpy="0 0 0"/>
+    </link>
+    <link name="${name}_mount_p">
+      <origin xyz="0 0 0" rpy="0 0 0"/>
+    </link>
+    <link name="${name}_rod">
       <visual>
+        <origin xyz="0 ${field_width/2} 0" rpy="0 ${pi/2} ${pi/2}"/>
         <geometry>
-          <cylinder length="${rod_length}" radius="${rod_diameter}/2"/>
+          <cylinder length="${rod_length}" radius="${rod_diameter/2}"/>
         </geometry>
-      </visual>
-  </xacro:macro>
-  <xacro:macro name="side_wall" params="side">
-    <link name="${name}_side_wall">
-      <visual>
-        <geometry>
-          <box size="${field_length} ${field_width} ${wall_height}"/>
-        </geometry>
+        <material name="Grey">
+          <color rgba="0.5 0.5 0.5 1"/>
+        </material>
       </visual>
     </link>
+    <joint name="${name}_mount_joint_c" type="fixed">
+      <origin xyz="${dir*dist} ${-field_width/2} ${rod_mountingheight}"/>
+      <parent link="field"/>
+      <child link="${name}_mount_c"/>
+    </joint>
+    <joint name="${name}_mount_joint_p" type="continuous">
+      <parent link="${name}_mount_c"/>
+      <child link="${name}_mount_p"/>
+      <axis xyz="0 1 0"/>
+    </joint>
+    <joint name="${name}_rod_joint_p" type="prismatic">
+      <origin xyz="0 0 0" rpy="0 0 0"/>
+      <parent link="${name}_mount_p"/>
+      <child link="${name}_rod"/>
+      <axis xyz="0 1 0"/>
+      <limit upper="0.05" lower="-0.05" effort="10" velocity="2"/>
+    </joint>
   </xacro:macro>
+  <!-- Macro to create the left and right wall panels -->
+  <xacro:macro name="side_wall" params="side dir">
+    <link name="${side}_side_wall">
+      <visual>
+        <origin xyz="0 ${dir*wall_thickness/2} ${wall_height/2}" rpy="0 0 0"/>
+        <geometry>
+          <box size="${field_length + wall_thickness*2} ${wall_thickness} ${wall_height}"/>
+        </geometry>
+        <material name="Soft Black">
+          <color rgba="0.1 0.1 0.1 1"/>
+        </material>
+      </visual>
+    </link>
+    <joint name="${side}_side_wall_joint" type="fixed">
+      <origin xyz="0 ${dir*field_width/2} 0" rpy="0 0 0" />
+      <parent link="field"/>
+      <child link="${side}_side_wall"/>
+    </joint>
+  </xacro:macro>
+  <!-- Macros to create the goal panels with a cut out for the goal -->
+  <xacro:macro name="end_wall" params="side dir">
+    <link name="${side}_end_wall_goal">
+      <visual>
+        <origin xyz="${dir*wall_thickness/2} 0 ${(wall_height+goal_height)/2}" rpy="0 0 0"/>
+        <geometry>
+          <box size="${wall_thickness} ${goal_width} ${wall_height-goal_height}"/>
+        </geometry>
+        <material name="Soft Black">
+          <color rgba="0.1 0.1 0.1 1"/>
+        </material>
+      </visual>
+    </link>
+    <joint name="${side}_end_wall_joint" type="fixed">
+      <origin xyz="${dir*field_length/2} 0 ${0}" rpy="0 0 0" />
+      <parent link="field"/>
+      <child link="${side}_end_wall_goal"/>
+    </joint>
+    <xacro:end_wall_segment end_color="${side}" end_dir="${dir}" side="right" dir="1"/>
+    <xacro:end_wall_segment end_color="${side}" end_dir="${dir}"  side="left" dir="-1"/>
+  </xacro:macro>
+  <xacro:macro name="end_wall_segment" params="end_color end_dir side dir">
+    <link name="${end_color}_end_wall_${side}">
+      <visual>
+        <origin xyz="${end_dir*wall_thickness/2} 0 ${wall_height/2}" rpy="0 0 0"/>
+        <geometry>
+          <box size="${wall_thickness} ${(field_width-goal_width)/2} ${wall_height}"/>
+        </geometry>
+        <material name="Soft Black">
+          <color rgba="0.1 0.1 0.1 1"/>
+        </material>
+      </visual>
+    </link>
+    <joint name="${end_color}_end_wall_${side}_joint" type="fixed">
+      <origin xyz="0 ${dir*(goal_width/2 + (field_width-goal_width)/4)} 0" rpy="0 0 0" />
+      <parent link="${end_color}_end_wall_goal"/>
+      <child link="${end_color}_end_wall_${side}"/>
+    </joint>
+  </xacro:macro>
+  <!-- START BUILD THE URDF MODEL -->
   <link name="base_link">
     <origin xyz="0 0 0" rpy="0 0 0"/>
@@ -50,4 +131,5 @@
   <link name="field">
     <visual>
+      <origin xyz="0 0 ${-field_thickness/2}" rpy="0 0 0"/>
       <geometry>
         <box size="${field_length} ${field_width} ${field_thickness}"/>
@@ -63,3 +145,11 @@
     <child link="field"/>
   </joint>
+  <xacro:side_wall side="right" dir="1"/>
+  <xacro:side_wall side="left" dir="-1"/>
+  <xacro:end_wall side="white" dir="1"/>
+  <xacro:end_wall side="grey" dir="-1"/>
+  <xacro:player_rod name="white_attack" dir="1" dist="${attack_rod_distance}" num_players="3" r="1" g="1" b="1"/>
+  <xacro:player_rod name="white_goalie" dir="-1" dist="${goalie_rod_distance}" num_players="3" r="1" g="1" b="1"/>
+  <xacro:player_rod name="grey_attack" dir="-1" dist="${attack_rod_distance}" num_players="3" r="1" g="1" b="1"/>
+  <xacro:player_rod name="grey_goalie" dir="1" dist="${goalie_rod_distance}" num_players="3" r="1" g="1" b="1"/>
 </robot>

Commit message: Finished table urdf, ball will be represented with tf broadcaster

File: table_description/urdf/table.urdf.xacro (robot description, xacro)
@@ -1,4 +1,4 @@
 <?xml version="1.0"?>
-<robot xmlns:xacro="http://www.ros.org/wiki/xacro" name="diff_drive">
+<robot xmlns:xacro="http://www.ros.org/wiki/xacro" name="table">
   <xacro:property name="props" value="${load_yaml('$(find table_description)/config/table_params.yaml')}"/>
   <xacro:property name="rod_length" value="${props['rod_length']}"/>
@@ -8,4 +8,5 @@
   <xacro:property name="player_depth" value="${props['player_depth']}"/>
   <xacro:property name="player_height" value="${props['player_height']}"/>
+  <xacro:property name="player_mountingheight" value="${props['rod_mountingheight']}"/>
   <xacro:property name="ball_diameter" value="${props['ball_diameter']}"/>
   <xacro:property name="field_width" value="${props['field_width']}"/>
@@ -19,17 +20,23 @@
   <xacro:property name="wall_thickness" value="0.015"/>
   <!-- Macro to create a player -->
-  <xacro:macro name="player" params="name r g b">
-    <link name="${name}">
-      <geometry>
-        <origin xyz="0 0 0" rpy="0 0 0"/>
-        <box size="${player_height} ${player_width} ${player_depth}"/>
-        <material name="White">
-          <color rgba="r g b 1.0"/>
+  <xacro:macro name="player" params="rod_name player_num r g b">
+    <link name="${rod_name}_player_${player_num}">
+      <visual>
+        <origin xyz="0 0 ${player_height/2 - player_mountingheight}" rpy="0 0 0"/>
+        <geometry>
+          <box size="${player_depth} ${player_width} ${player_height}"/>
+        </geometry>
+        <material name="${rod_name}">
+          <color rgba="${r} ${g} ${b} 1.0"/>
         </material>
-      </geometry>
+      </visual>
     </link>
+    <joint name="${rod_name}_player_${player_num}_joint" type="fixed">
+      <parent link="${name}_p${player_num}_mount"/>
+      <child link="${rod_name}_player_${player_num}"/>
+    </joint>
   </xacro:macro>
   <!-- Macro to create a player rod -->
-  <xacro:macro name="player_rod" params="name dir dist num_players r g b">
+  <xacro:macro name="player_rod" params="name dir dist r g b">
     <link name="${name}_mount_c">
       <origin xyz="0 0 0" rpy="0 0 0"/>
@@ -66,4 +73,26 @@
       <limit upper="0.05" lower="-0.05" effort="10" velocity="2"/>
     </joint>
+    <!-- attach players to each rod -->
+    <link name="${name}_p1_mount"/>
+    <link name="${name}_p2_mount"/>
+    <link name="${name}_p3_mount"/>
+    <joint name="${name}_p1_mount_joint" type="fixed">
+      <origin xyz="0 0.061 0" rpy="0 0 0"/>
+      <parent link="${name}_rod"/>
+      <child link="${name}_p1_mount"/>
+    </joint>
+    <joint name="${name}_p2_mount_joint" type="fixed">
+      <origin xyz="0 0.141 0" rpy="0 0 0"/>
+      <parent link="${name}_rod"/>
+      <child link="${name}_p2_mount"/>
+    </joint>
+    <joint name="${name}_p3_mount_joint" type="fixed">
+      <origin xyz="0 0.221 0" rpy="0 0 0"/>
+      <parent link="${name}_rod"/>
+      <child link="${name}_p3_mount"/>
+    </joint>
+    <xacro:player rod_name="${name}" player_num="1" r="${r}" g="${g}" b="${b}"/>
+    <xacro:player rod_name="${name}" player_num="2" r="${r}" g="${g}" b="${b}"/>
+    <xacro:player rod_name="${name}" player_num="3" r="${r}" g="${g}" b="${b}"/>
   </xacro:macro>
   <!-- Macro to create the left and right wall panels -->
@@ -125,5 +154,5 @@
     </joint>
   </xacro:macro>
-  <!-- START BUILD THE URDF MODEL -->
+  <!-- START BUILDING THE URDF MODEL -->
   <link name="base_link">
     <origin xyz="0 0 0" rpy="0 0 0"/>
@@ -149,7 +178,7 @@
   <xacro:end_wall side="white" dir="1"/>
   <xacro:end_wall side="grey" dir="-1"/>
-  <xacro:player_rod name="white_attack" dir="1" dist="${attack_rod_distance}" num_players="3" r="1" g="1" b="1"/>
-  <xacro:player_rod name="white_goalie" dir="-1" dist="${goalie_rod_distance}" num_players="3" r="1" g="1" b="1"/>
-  <xacro:player_rod name="grey_attack" dir="-1" dist="${attack_rod_distance}" num_players="3" r="1" g="1" b="1"/>
-  <xacro:player_rod name="grey_goalie" dir="1" dist="${goalie_rod_distance}" num_players="3" r="1" g="1" b="1"/>
+  <xacro:player_rod name="white_attack" dir="1" dist="${attack_rod_distance}" r="1" g="1" b="1"/>
+  <xacro:player_rod name="white_goalie" dir="-1" dist="${goalie_rod_distance}" r="1" g="1" b="1"/>
+  <xacro:player_rod name="grey_attack" dir="-1" dist="${attack_rod_distance}" r="0.5" g="0.5" b="0.5"/>
+  <xacro:player_rod name="grey_goalie" dir="1" dist="${goalie_rod_distance}" r="0.5" g="0.5" b="0.5"/>
 </robot>

Commit message: hacked together accurate ball position estimation, integrating with the motors

File: table_description/urdf/table.urdf.xacro (robot description, xacro)
@@ -18,4 +18,5 @@
   <xacro:property name="attack_rod_distance" value="${props['attack_rod_distance']}"/>
   <xacro:property name="goalie_rod_distance" value="${props['goalie_rod_distance']}"/>
+  <xacro:property name="rod_travel_distance" value="${props['rod_travel_distance']}"/>
   <xacro:property name="wall_thickness" value="0.015"/>
   <!-- Macro to create a player -->
@@ -71,5 +72,5 @@
       <child link="${name}_rod"/>
       <axis xyz="0 1 0"/>
-      <limit upper="0.05" lower="-0.05" effort="10" velocity="2"/>
+      <limit upper="${rod_travel_distance/2}" lower="${-rod_travel_distance/2}" effort="10" velocity="2"/>
     </joint>
     <!-- attach players to each rod -->

Commit message: Functioning linear position command, need account for error cases and incorperate hysteresis

File: table_description/urdf/table.urdf.xacro (robot description, xacro)
@@ -57,15 +57,15 @@
       </visual>
     </link>
-    <joint name="${name}_mount_joint_c" type="fixed">
+    <joint name="${name}_fixed_joint" type="fixed">
       <origin xyz="${dir*dist} ${-field_width/2} ${rod_mountingheight}"/>
       <parent link="field"/>
       <child link="${name}_mount_c"/>
     </joint>
-    <joint name="${name}_mount_joint_p" type="continuous">
+    <joint name="${name}_rot_joint" type="continuous">
       <parent link="${name}_mount_c"/>
       <child link="${name}_mount_p"/>
       <axis xyz="0 1 0"/>
     </joint>
-    <joint name="${name}_rod_joint_p" type="prismatic">
+    <joint name="${name}_lin_joint" type="prismatic">
       <origin xyz="0 0 0" rpy="0 0 0"/>
       <parent link="${name}_mount_p"/>

Commit message: Table working! need to clean up code base

File: table_description/urdf/table.urdf.xacro (robot description, xacro)
@@ -59,5 +59,5 @@
     <joint name="${name}_fixed_joint" type="fixed">
       <origin xyz="${dir*dist} ${-field_width/2} ${rod_mountingheight}"/>
-      <parent link="field"/>
+      <parent link="table_base"/>
       <child link="${name}_mount_c"/>
     </joint>
@@ -112,5 +112,5 @@
     <joint name="${side}_side_wall_joint" type="fixed">
       <origin xyz="0 ${dir*field_width/2} 0" rpy="0 0 0" />
-      <parent link="field"/>
+      <parent link="table_base"/>
       <child link="${side}_side_wall"/>
     </joint>
@@ -131,5 +131,5 @@
     <joint name="${side}_end_wall_joint" type="fixed">
       <origin xyz="${dir*field_length/2} 0 ${0}" rpy="0 0 0" />
-      <parent link="field"/>
+      <parent link="table_base"/>
       <child link="${side}_end_wall_goal"/>
     </joint>
@@ -159,5 +159,5 @@
     <origin xyz="0 0 0" rpy="0 0 0"/>
   </link>
-  <link name="field">
+  <link name="table_base">
     <visual>
       <origin xyz="0 0 ${-field_thickness/2}" rpy="0 0 0"/>
@@ -170,6 +170,14 @@
     </visual>
   </link>
+  <joint name="table_base_joint" type="fixed">
+    <origin xyz="0 0 0" rpy="0 0 0" />
+    <parent link="base_link"/>
+    <child link="table_base"/>
+  </joint>
+  <link name="field">
+    <origin xyz="0 0 0" rpy="0 0 0"/>
+  </link>
   <joint name="field_joint" type="fixed">
-    <origin xyz="0 0 0" rpy="0 0 0" />
+    <origin xyz="${(-field_length + ball_diameter)/2} ${(-field_width + ball_diameter)/2} 0" rpy="0 0 0" />
     <parent link="base_link"/>
     <child link="field"/>
